File: Arduino Micro RGB Controller/Arduino Micro RGB Controller.brd (EAGLE design)
At the start: 58.4 x 31.4 mm, 43 parts, among them IC1 REG1117, Q4 220mA/50V/3.5Ω, Q5 220mA/50V/3.5Ω, U1 32U4, X1 16Mhz

Commit message: Add files via upload
Parts:
- added C13: 100nF, adafruit:C0805
Connections:
- new net N$9: C13.2, U1.42
- net GND: now also C13.1
Routing:
- net N$9: track 0.00 -> 14.7 mm, vias 0 -> 2
Changed lines of the file:
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@@
 <element name="R4" library="adafruit" package="M0805" value="10k" x="49.784" y="12.192" smashed="yes" rot="R180"/>
 <element name="R5" library="adafruit" package="M0805" value="10k" x="54.102" y="23.876" smashed="yes" rot="R180"/>
-<element name="R6" library="adafruit" package="M0805" value="10k" x="51.562" y="19.05" smashed="yes" rot="R90">
-<attribute name="NAME" x="50.546" y="18.034" size="1.27" layer="25" rot="R90"/>
-</element>
+<element name="R6" library="adafruit" package="M0805" value="10k" x="51.562" y="19.05" smashed="yes" rot="R90"/>
 <element name="R7" library="adafruit" package="M0805" value="10k" x="49.276" y="19.05" smashed="yes" rot="R270"/>
 <element name="RGBLED" library="pinhead" library_urn="urn:adsk.eagle:library:325" package="1X04" package3d_urn="urn:adsk.eagle:package:22407/2" value="RGBLED" x="19.05" y="27.94" smashed="yes"/>
@@
 <attribute name="VALUE" x="17.991" y="27.065" size="1.27" layer="27" rot="R180"/>
 </element>
+<element name="C13" library="adafruit" package="C0805" value="100nF" x="21.844" y="9.525" smashed="yes"/>
 </elements>
 <signals>
@@
 <wire x1="4.732" y1="5.05" x2="5.872" y2="5.05" width="0.508" layer="1"/>
 <wire x1="5.872" y1="5.05" x2="6.096" y2="4.826" width="0.508" layer="1"/>
+<contactref element="C13" pad="1"/>
 </signal>
 <signal name="VOUT">
@@
 <wire x1="12.2386625" y1="3.5236" x2="19.7453375" y2="3.5236" width="0.508" layer="1"/>
 </signal>
+<signal name="N$9">
+<contactref element="C13" pad="2"/>
+<contactref element="U1" pad="42"/>
+<wire x1="32.3" y1="11.57" x2="32.004" y2="11.274" width="0.2032" layer="1"/>
+<wire x1="32.004" y1="11.274" x2="31.4447875" y2="11.274" width="0.2032" layer="1"/>
+<wire x1="31.103" y1="8.6817875" x2="30.988" y2="8.5667875" width="0.2032" layer="1"/>
+<wire x1="30.988" y1="8.5667875" x2="30.988" y2="7.747" width="0.2032" layer="1"/>
+<wire x1="31.4447875" y1="11.274" x2="31.103" y2="10.9322125" width="0.2032" layer="1"/>
+<wire x1="31.103" y1="10.9322125" x2="31.103" y2="8.6817875" width="0.2032" layer="1"/>
+<wire x1="30.988" y1="7.747" x2="28.956" y2="7.747" width="0.2032" layer="1"/>
+<wire x1="28.956" y1="7.747" x2="28.702" y2="8.001" width="0.2032" layer="1"/>
+<via x="28.702" y="8.001" extent="1-16" drill="0.35"/>
+<wire x1="28.702" y1="8.001" x2="26.035" y2="10.668" width="0.2032" layer="16"/>
+<wire x1="26.035" y1="10.668" x2="25.019" y2="10.668" width="0.2032" layer="16"/>
+<via x="25.019" y="10.668" extent="1-16" drill="0.35"/>
+<wire x1="25.019" y1="10.668" x2="24.13506875" y2="10.668" width="0.2032" layer="1"/>
+<wire x1="24.13506875" y1="10.668" x2="24.01086875" y2="10.5438" width="0.2032" layer="1"/>
+<wire x1="24.01086875" y1="10.5438" x2="23.7128" y2="10.5438" width="0.2032" layer="1"/>
+<wire x1="23.7128" y1="10.5438" x2="22.694" y2="9.525" width="0.2032" layer="1"/>
+</signal>
 </signals>
