File: Arduino Micro RGB Controller/Arduino Micro RGB Controller.sch (EAGLE design)
At the start: 43 parts, among them IC1 REG1117, Q4 220mA/50V/3.5Ω, Q5 220mA/50V/3.5Ω, U1 32U4, X1 16Mhz

Commit message: Add files via upload
Parts:
- added C13: 100nF, adafruit:C-USC0805
Connections:
- new net N$9: C13.2, U1.AREF
- net GND: now also C13.1
Changed lines of the file:
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@@
 <part name="LED3" library="adafruit" deviceset="LED" device="CHIPLED_0603"/>
 <part name="D3" library="diode" library_urn="urn:adsk.eagle:library:210" deviceset="DIODE-" device="SOD123" package3d_urn="urn:adsk.eagle:package:43420/1"/>
+<part name="C13" library="adafruit" deviceset="C-US" device="C0805" value="100nF"/>
 </parts>
 <sheets>
@@
 <instance part="LED3" gate="G$1" x="238.76" y="93.98"/>
 <instance part="D3" gate="G$1" x="167.64" y="116.84"/>
+<instance part="C13" gate="G$1" x="114.3" y="68.58" rot="R90"/>
 </instances>
 <busses>
@@
 <junction x="78.74" y="73.66"/>
 <pinref part="GND6" gate="1" pin="GND"/>
+<pinref part="C13" gate="G$1" pin="1"/>
+<wire x1="111.76" y1="68.58" x2="109.22" y2="68.58" width="0.1524" layer="91"/>
+<wire x1="109.22" y1="68.58" x2="109.22" y2="73.66" width="0.1524" layer="91"/>
+<junction x="109.22" y="73.66"/>
 </segment>
 <segment>
@@
 </segment>
 </net>
+<net name="N$9" class="0">
+<segment>
+<pinref part="C13" gate="G$1" pin="2"/>
+<pinref part="U1" gate="U1" pin="AREF"/>
+<wire x1="119.38" y1="68.58" x2="119.38" y2="73.66" width="0.1524" layer="91"/>
+<wire x1="119.38" y1="73.66" x2="134.62" y2="73.66" width="0.1524" layer="91"/>
+</segment>
+</net>
